File: 電源基板/電源基板.kicad_sch (KiCad schematic)
At the start: 16 parts, among them J1 Conn_01x02, J2 Conn_01x02, J3 Conn_01x02, J4 Conn_01x02, J5 Conn_01x02, SW1 SW_SPST

Commit message: 5V生成をLDOからDCDCに
Parts:
- removed C1: 22uF, symbol Device:C_Polarized
- removed C2: 0.33uF, symbol Device:C_Polarized
- removed NJM2396F2: ~, symbol NJM2396F05:NJM2396F05
- added C5: 22uF, symbol Device:C
- added C6: 10uF, symbol Device:C
- added J6: 01x02_Pin, symbol Connector:Conn_01x02_Pin
- added J7: Conn_01x02_ToF_Camera, symbol Connector_Generic:Conn_01x02
- added PS1: OKL-T_6-W12N-C, OKLT6W12NC, symbol OKL-T_6-W12N-C:OKL-T_6-W12N-C
- added R1: 20k, symbol Device:R
- added R2, R3: 1.2k, symbol Device:R
- added RV1: 20k, symbol Device:R_Potentiometer
Connections:
- net +5V: now also C6.1, J7.1 (Pin_1), PS1.4 (VOUT), PS1.5 (SENSE), R2.1
- net 6.6V: now also C5.2, PS1.2 (VIN), R1.2
- net GND: now also C5.1, C6.2, J6.2 (Pin_2), J7.2 (Pin_2), PS1.3 (GROUND_1), PS1.7 (GROUND_2), R2.2, R3.2
- new net: PS1.6 (TRIM), RV1.1
- new net: R3.1, RV1.2, RV1.3
- new net: J6.1 (Pin_1), PS1.1 (ON/OFF_CONTROL), R1.1
- no-connect marks 8 -> 13
Other:
- company: (none) -> Koki
- title: (none) -> 電源基板
